Commit message: Added pocketbot link to robot model

File: docker_ros_nodes/description/model.urdf.xacro (robot description, xacro)
@@ -66,5 +66,5 @@
     <parent link="base_link"/>
     <child link="scanmatcher_frame"/>
-    <origin rpy="0 0 0" xyz="0 0 0"/>
+    <origin rpy="0 0 0" xyz="0 0 0.1"/>
   </joint>
     <link name="scanmatcher_frame">
@@ -78,3 +78,19 @@
     </visual>
   </link>
+    <joint name="imu_joint" type="fixed">
+    <axis xyz="0 0 0"/>
+    <parent link="base_link"/>
+    <child link="pocketbot"/>
+    <origin rpy="0 0 0.0" xyz="0 0 0.1"/>
+  </joint>
+    <link name="pocketbot">
+    <visual>
+      <geometry>
+        <box size="0.1 0.1 0.1"/>
+      </geometry>
+      <material name="green">
+	      <color rgba="0.1 0.8 0.1 1"/>
+	    </material>
+    </visual>
+  </link>
 </robot>

Commit message: Added gazebo simulation

File: docker_ros_nodes/description/model.urdf.xacro (robot description, xacro)
@@ -5,8 +5,14 @@
        xmlns:interface="http://playerstage.sourceforge.net/gazebo/xmlschema/#interface"
        xmlns:xacro="http://ros.org/wiki/xacro">
+  <xacro:property name="wheel_length" value="0.005" />
+  <xacro:property name="wheel_radius" value="0.05" />
+  <xacro:property name="body_length" value="0.4" />
+  <xacro:property name="body_width" value="0.3" />
+  <xacro:property name="body_height" value="0.15" />
+  <xacro:property name="laser_size" value="0.1" />
   <link name="base_link">
     <visual>
       <geometry>
-        <box size="0.2 0.1 0.1"/>
+        <box size="${body_length} ${body_width} ${body_height}"/>
       </geometry>
       <material name="blue">
@@ -16,44 +22,23 @@
     <collision>
       <geometry>
-        <box size="0.2 0.1 0.1"/>
+        <box size="${body_width} ${body_length} ${body_height}"/>
       </geometry>
     </collision>
-  </link>
- <!-- <joint name="center_joint" type="fixed">-->
- <!--   <axis xyz="0 0 1"/>-->
- <!--   <parent link="device"/>-->
- <!--   <child link="base_link"/>-->
- <!--   <origin rpy="0 0 0" xyz="0 0 0.2"/>-->
- <!-- </joint>-->
- <!-- <link name="device">-->
- <!--   <visual>-->
- <!--     <geometry>-->
- <!--       <box size="0.41148 0.30988 0.05588"/>-->
- <!--     </geometry>-->
- <!--     <material name="black">-->
-	<!--<color rgba="0.0 0.0 0.0 1"/>-->
- <!--     </material>-->
- <!--   </visual>-->
- <!--   <collision>-->
- <!--     <geometry>-->
- <!--       <box size="0.41148 0.30988 0.05588"/>-->
- <!--     </geometry>-->
- <!--   </collision>-->
- <!--  <inertial>-->
- <!--     <mass value="20.0"/>-->
- <!--     <inertia ixx="1.0" iyy="1.0" izz="1.0"-->
- <!--              ixy="0" ixz="0" iyz="0"/>-->
- <!--   </inertial>-->
- <!-- </link>-->
+    <inertial>
+      <mass value="20"/>
+      <inertia ixx="0.01" iyy="0.01" izz="0.01"
+               ixy="0" ixz="0" iyz="0"/>
+    </inertial>
+  </link>
   <joint name="laser_joint" type="fixed">
     <axis xyz="0 0 0"/>
     <parent link="base_link"/>
     <child link="laser"/>
-    <origin rpy="0 0 0" xyz="0 0 0"/>
+    <origin rpy="0 0 0" xyz="0 0 ${body_height / 2 + laser_size / 2}"/>
   </joint>
   <link name="laser">
     <visual>
       <geometry>
-        <box size="0.1 0.1 0.1"/>
+        <box size="${laser_size} ${laser_size} ${laser_size}"/>
       </geometry>
       <material name="purple">
@@ -61,4 +46,9 @@
 	    </material>
     </visual>
+    <inertial>
+      <mass value="0.1"/>
+      <inertia ixx="0.001" iyy="0.001" izz="0.001"
+               ixy="0" ixz="0" iyz="0"/>
+    </inertial>
   </link>
   <joint name="odom_joint" type="fixed">
@@ -68,5 +58,5 @@
     <origin rpy="0 0 0" xyz="0 0 0.1"/>
   </joint>
-    <link name="scanmatcher_frame">
+  <link name="scanmatcher_frame">
     <visual>
       <geometry>
@@ -77,4 +67,9 @@
 	    </material>
     </visual>
+    <inertial>
+      <mass value="0.01"/>
+      <inertia ixx="0.001" iyy="0.001" izz="0.001"
+               ixy="0" ixz="0" iyz="0"/>
+    </inertial>
   </link>
     <joint name="imu_joint" type="fixed">
@@ -93,4 +88,136 @@
 	    </material>
     </visual>
-  </link>
+    <inertial>
+      <mass value="0.01"/>
+      <inertia ixx="0.001" iyy="0.001" izz="0.001"
+               ixy="0" ixz="0" iyz="0"/>
+    </inertial>
+  </link>
+  <link name="wheel_right">
+      <visual>
+        <geometry>
+          <cylinder length="${wheel_length}" radius="${wheel_radius}"/>
+        </geometry>
+        <material name="black"/>
+      </visual>
+      <collision>
+        <geometry>
+          <cylinder length="${wheel_length}" radius="${wheel_radius}"/>
+        </geometry>
+      </collision>
+      <inertial>
+        <mass value="0.01"/>
+        <inertia ixx="1.0" iyy="1.0" izz="1.0"
+                 ixy="0" ixz="0" iyz="0"/>
+      </inertial>
+    </link>
+    <joint name="axis_right" type="continuous">
+      <axis xyz="0 0 1"/>
+      <parent link="base_link"/>
+      <child link="wheel_right"/>
+      <origin rpy="-1.5708 0 0" xyz="-${body_length / 2 - wheel_radius * 2} ${body_width / 2 + wheel_length} -${body_height / 2 - wheel_radius + wheel_length}"/>
+    </joint>
+    <link name="wheel_left">
+      <visual>
+        <geometry>
+          <cylinder length="${wheel_length}" radius="${wheel_radius}"/>
+        </geometry>
+        <material name="black"/>
+      </visual>
+      <collision>
+        <geometry>
+          <cylinder length="${wheel_length}" radius="${wheel_radius}"/>
+        </geometry>
+      </collision>
+      <inertial>
+        <mass value="0.01"/>
+        <inertia ixx="1.0" iyy="1.0" izz="1.0"
+                 ixy="0" ixz="0" iyz="0"/>
+      </inertial>
+      <gazebo reference="wheel_left">
+        <material>Gazebo/Black</material>
+      </gazebo>
+    </link>
+    <joint name="axis_left" type="continuous">
+      <axis xyz="0 0 1"/>
+      <parent link="base_link"/>
+      <child link="wheel_left"/>
+      <origin rpy="-1.5708 0 0" xyz="-${body_length / 2 - wheel_radius * 2} -${body_width / 2 + wheel_length} -${body_height / 2 - wheel_radius + wheel_length}"/>
+    </joint>
+    <link name="caster">
+      <visual>
+        <geometry>
+          <sphere radius="${wheel_radius}"/>
+        </geometry>
+        <material name="black"/>
+      </visual>
+      <collision>
+        <geometry>
+          <sphere radius="${wheel_radius}"/>
+        </geometry>
+      </collision>
+      <inertial>
+        <mass value="0.01"/>
+        <inertia ixx="0.001" iyy="0.001" izz="0.001"
+                 ixy="0" ixz="0" iyz="0"/>
+      </inertial>
+    </link>
+    <joint name="axis_caster" type="fixed">
+      <axis xyz="1 1 1"/>
+      <parent link="base_link"/>
+      <child link="caster"/>
+      <origin rpy="0 0 0" xyz="${body_length / 2 - wheel_radius * 2} 0 -${body_height / 2 - wheel_radius + wheel_length}"/>
+    </joint>
+<!-- Gazebo Drivers -->
+  <gazebo reference="laser">
+    <material>Gazebo/Blue</material>
+    <sensor type="ray" name="laser_sensor">
+      <pose>0 0 0 0 0 0</pose>
+      <visualize>true</visualize>
+      <update_rate>40</update_rate>
+      <ray>
+        <scan>
+          <horizontal>
+            <samples>720</samples>
+            <resolution>1</resolution>
+            <min_angle>-1.570795</min_angle>
+            <max_angle>1.570795</max_angle>
+          </horizontal>
+        </scan>
+        <range>
+          <min>0.10</min>
+          <max>30.0</max>
+          <resolution>0.01</resolution>
+        </range>
+        <noise>
+          <type>gaussian</type>
+          <!-- Noise parameters based on published spec for Hokuyo laser
+               achieving "+-30mm" accuracy at range < 10m.  A mean of 0.0m and
+               stddev of 0.01m will put 99.7% of samples within 0.03m of the true
+               reading. -->
+          <mean>0.0</mean>
+          <stddev>0.01</stddev>
+        </noise>
+      </ray>
+      <plugin name="gazebo_ros_head_hokuyo_controller" filename="libgazebo_ros_laser.so">
+        <topicName>/scan</topicName>
+        <frameName>laser</frameName>
+      </plugin>
+    </sensor>
+  </gazebo>
+  <gazebo>
+    <plugin name="differential_drive_controller" filename="libgazebo_ros_diff_drive.so">
+      <alwaysOn>true</alwaysOn>
+      <updateRate>20</updateRate>
+      <leftJoint>axis_left</leftJoint>
+      <rightJoint>axis_right</rightJoint>
+      <wheelSeparation>0.254</wheelSeparation>
+      <wheelDiameter>0.1524</wheelDiameter>
+      <torque>100</torque>
+      <commandTopic>cmd_vel</commandTopic>
+      <odometryTopic>odom</odometryTopic>
+      <odometryFrame>odom</odometryFrame>
+      <robotBaseFrame>base_link</robotBaseFrame>
+    </plugin>
+  </gazebo>
 </robot>

Commit message: Hector mapping updated for x86

File: docker_ros_nodes/description/model.urdf.xacro (robot description, xacro)
@@ -52,35 +52,14 @@
     </inertial>
   </link>
-  <joint name="odom_joint" type="fixed">
-    <axis xyz="0 0 0"/>
-    <parent link="base_link"/>
-    <child link="scanmatcher_frame"/>
-    <origin rpy="0 0 0" xyz="0 0 0.1"/>
-  </joint>
-  <link name="scanmatcher_frame">
-    <visual>
-      <geometry>
-        <box size="0.1 0.1 0.1"/>
-      </geometry>
-      <material name="red">
-	      <color rgba="0.5 0.0 0.1 1"/>
-	    </material>
-    </visual>
-    <inertial>
-      <mass value="0.01"/>
-      <inertia ixx="0.001" iyy="0.001" izz="0.001"
-               ixy="0" ixz="0" iyz="0"/>
-    </inertial>
-  </link>
-    <joint name="imu_joint" type="fixed">
+  <joint name="imu_joint" type="fixed">
     <axis xyz="0 0 0"/>
     <parent link="base_link"/>
     <child link="pocketbot"/>
-    <origin rpy="0 0 0.0" xyz="0 0 0.1"/>
+    <origin rpy="0 0 0.0" xyz="0 0 ${laser_size * 2}"/>
   </joint>
-    <link name="pocketbot">
+  <link name="pocketbot">
     <visual>
       <geometry>
-        <box size="0.1 0.1 0.1"/>
+        <box size="${laser_size} ${laser_size} ${laser_size}"/>
       </geometry>
       <material name="green">

Commit message: Improved robot model

File: docker_ros_nodes/description/model.urdf.xacro (robot description, xacro)
@@ -5,6 +5,6 @@
        xmlns:interface="http://playerstage.sourceforge.net/gazebo/xmlschema/#interface"
        xmlns:xacro="http://ros.org/wiki/xacro">
-  <xacro:property name="wheel_length" value="0.005" />
-  <xacro:property name="wheel_radius" value="0.05" />
+  <xacro:property name="wheel_length" value="0.02" />
+  <xacro:property name="wheel_radius" value="0.0725" />
   <xacro:property name="body_length" value="0.4" />
   <xacro:property name="body_width" value="0.3" />

Commit message: Model now working with Gazebo

File: docker_ros_nodes/description/model.urdf.xacro (robot description, xacro)
@@ -7,8 +7,11 @@
   <xacro:property name="wheel_length" value="0.02" />
   <xacro:property name="wheel_radius" value="0.0725" />
-  <xacro:property name="body_length" value="0.4" />
+  <xacro:property name="body_length" value="0.3" />
   <xacro:property name="body_width" value="0.3" />
   <xacro:property name="body_height" value="0.15" />
   <xacro:property name="laser_size" value="0.1" />
+  <xacro:property name="wheel_x" value="-${body_length / 2 - wheel_radius}" />
+  <xacro:property name="wheel_y" value="-${body_width / 2 - wheel_length}" />
+  <xacro:property name="wheel_inertia" value="0.01" />
   <link name="base_link">
     <visual>
@@ -20,11 +23,11 @@
       </material>
     </visual>
-    <collision>
+    <!--<collision>
       <geometry>
         <box size="${body_width} ${body_length} ${body_height}"/>
       </geometry>
-    </collision>
+    </collision>-->
     <inertial>
-      <mass value="20"/>
+      <mass value="5"/>
       <inertia ixx="0.01" iyy="0.01" izz="0.01"
                ixy="0" ixz="0" iyz="0"/>
@@ -87,5 +90,5 @@
       <inertial>
         <mass value="0.01"/>
-        <inertia ixx="1.0" iyy="1.0" izz="1.0"
+        <inertia ixx="${wheel_inertia}" iyy="${wheel_inertia}" izz="${wheel_inertia}"
                  ixy="0" ixz="0" iyz="0"/>
       </inertial>
@@ -95,5 +98,5 @@
       <parent link="base_link"/>
       <child link="wheel_right"/>
-      <origin rpy="-1.5708 0 0" xyz="-${body_length / 2 - wheel_radius * 2} ${body_width / 2 + wheel_length} -${body_height / 2 - wheel_radius + wheel_length}"/>
+      <origin rpy="-1.5708 0 0" xyz="${wheel_x} ${-wheel_y} -${body_height / 2 - wheel_radius + wheel_length}"/>
     </joint>
     <link name="wheel_left">
@@ -111,5 +114,5 @@
       <inertial>
         <mass value="0.01"/>
-        <inertia ixx="1.0" iyy="1.0" izz="1.0"
+        <inertia ixx="${wheel_inertia}" iyy="${wheel_inertia}" izz="${wheel_inertia}"
                  ixy="0" ixz="0" iyz="0"/>
       </inertial>
@@ -122,5 +125,5 @@
       <parent link="base_link"/>
       <child link="wheel_left"/>
-      <origin rpy="-1.5708 0 0" xyz="-${body_length / 2 - wheel_radius * 2} -${body_width / 2 + wheel_length} -${body_height / 2 - wheel_radius + wheel_length}"/>
+      <origin rpy="-1.5708 0 0" xyz="${wheel_x} ${wheel_y} -${body_height / 2 - wheel_radius + wheel_length}"/>
     </joint>
     <link name="caster">
@@ -135,16 +138,24 @@
           <sphere radius="${wheel_radius}"/>
         </geometry>
+        <surface>
+          <friction>
+            <ode>
+              <mu>0.0</mu>
+              <mu2>0.0</mu2>
+            </ode>
+          </friction>
+        </surface>
       </collision>
       <inertial>
         <mass value="0.01"/>
-        <inertia ixx="0.001" iyy="0.001" izz="0.001"
+        <inertia ixx="${wheel_inertia}" iyy="${wheel_inertia}" izz="${wheel_inertia}"
                  ixy="0" ixz="0" iyz="0"/>
       </inertial>
     </link>
-    <joint name="axis_caster" type="fixed">
-      <axis xyz="1 1 1"/>
+    <joint name="axis_caster" type="continuous">
+      <axis xyz="0 0 1"/>
       <parent link="base_link"/>
       <child link="caster"/>
-      <origin rpy="0 0 0" xyz="${body_length / 2 - wheel_radius * 2} 0 -${body_height / 2 - wheel_radius + wheel_length}"/>
+      <origin rpy="-1.57079632679 0 0" xyz="${-1 * wheel_x} 0 -${body_height / 2 - wheel_radius + wheel_length}"/>
     </joint>
 <!-- Gazebo Drivers -->
@@ -153,5 +164,5 @@
     <sensor type="ray" name="laser_sensor">
       <pose>0 0 0 0 0 0</pose>
-      <visualize>true</visualize>
+      <visualize>false</visualize>
       <update_rate>40</update_rate>
       <ray>

Commit message: Added gmapping

File: docker_ros_nodes/description/model.urdf.xacro (robot description, xacro)
@@ -49,9 +49,4 @@
 	    </material>
     </visual>
-    <inertial>
-      <mass value="0.1"/>
-      <inertia ixx="0.001" iyy="0.001" izz="0.001"
-               ixy="0" ixz="0" iyz="0"/>
-    </inertial>
   </link>
   <joint name="imu_joint" type="fixed">
@@ -164,5 +159,5 @@
     <sensor type="ray" name="laser_sensor">
       <pose>0 0 0 0 0 0</pose>
-      <visualize>false</visualize>
+      <visualize>true</visualize>
       <update_rate>40</update_rate>
       <ray>
@@ -209,4 +204,15 @@
       <odometryFrame>odom</odometryFrame>
       <robotBaseFrame>base_link</robotBaseFrame>
+      <publishTf>1</publishTf>
+    </plugin>
+  </gazebo>
+  <gazebo>
+    <plugin name="imu_plugin" filename="libgazebo_ros_imu.so">
+      <alwaysOn>true</alwaysOn>
+      <bodyName>pocketbot</bodyName>
+      <topicName>imu</topicName>
+      <serviceName>imu_service</serviceName>
+      <gaussianNoise>0.0</gaussianNoise>
+      <updateRate>20.0</updateRate>
     </plugin>
   </gazebo>
