Commit message: Fixed alvar

File: docker_ros_nodes/ros-mars-rover-description/model.urdf (robot description, URDF)
Before this commit: robot efim, 9 links, 8 joints
Links:
- link body_link: geometry visual mesh filename=http://localhost:8888/rover.stl scale=0.015 0.015 0.015

File: docker_ros_nodes/ros-mars-rover-description/model.urdf.xacro (robot description, xacro)
@@ -28,6 +28,6 @@
     <visual>
       <geometry>
-        <cylinder length="1.04775" radius="0.2032"/>
-        <!-- <mesh filename="http://localhost:8888/rover.stl" scale="0.015 0.015 0.015"/> -->
+        <!-- <cylinder length="1.04775" radius="0.2032"/> -->
+        <mesh filename="http://localhost:8888/rover.stl" scale="0.015 0.015 0.015"/>
       </geometry>
       <!-- <material name="clear">
@@ -207,5 +207,5 @@
       <wheelDiameter>0.1524</wheelDiameter>
       <torque>20</torque>
-      <commandTopic>pocketbot/cmd_vel</commandTopic>
+      <commandTopic>cmd_vel</commandTopic>
       <odometryTopic>odom</odometryTopic>
       <odometryFrame>map</odometryFrame>
