Commit message: Added gzweb

File: docker_ros_nodes/ros-mars-rover-description/model.urdf.xacro (robot description, xacro)
@@ -22,370 +22,3 @@
     </inertial>
   </link>
-  <gazebo reference="base_link">
-    <material>Gazebo/Black</material>
-  </gazebo>
-  <link name="body_link">
-    <visual>
-      <geometry>
-        <!-- <cylinder length="1.04775" radius="0.2032"/> -->
-        <mesh filename="http://localhost:8888/rover.stl" scale="0.015 0.015 0.015"/>
-      </geometry>
-      <!-- <material name="clear">
-        <color rgba="0.75 0.75 0.75 0.4"/>
-      </material> -->
-      <material name="clear">
-        <color rgba="0.75 0.5 1.0 1.0"/>
-      </material>
-    </visual>
-    <!--<collision>
-      <geometry>
-        <cylinder length="1.04775" radius="0.2032"/>
-      </geometry>
-    </collision>-->
-    <inertial>
-      <mass value="10.0"/>
-      <inertia ixx="1.0" iyy="1.0" izz="1.0"
-               ixy="0" ixz="0" iyz="0"/>
-    </inertial>
-  </link>
-  <joint name="center_joint" type="fixed">
-    <axis xyz="0 0 1"/>
-    <parent link="base_link"/>
-    <child link="body_link"/>
-    <origin rpy="0 0 0" xyz="0 0 0.551815"/>
-  </joint>
-  <link name="camera_link">
-    <visual>
-      <origin rpy="0 0 0"/>
-      <geometry>
-        <box size="0.0762 0.2794 0.0762"/>
-      </geometry>
-      <material name="red">
-	<color rgba="1 0.1 0.1 1"/>
-      </material>
-    </visual>
-    <!--<collision>
-      <geometry>
-        <box size="0.0762 0.2794 0.0762"/>
-      </geometry>
-    </collision>-->
-   <inertial>
-      <mass value="0.25"/>
-      <inertia ixx="1.0" iyy="1.0" izz="1.0"
-               ixy="0" ixz="0" iyz="0"/>
-    </inertial>
-  </link>
-  <joint name="camera_joint" type="fixed">
-    <axis xyz="0 0 0"/>
-    <parent link="body_link"/>
-    <child link="camera_link"/>
-    <origin rpy="0 0 0" xyz="0.15 0 -0.25"/>
-  </joint>
-    <!-- The fixed joints & links below are usually published by static_transformers launched by the OpenNi launch
-         files. However, for Gazebo simulation we need them, so we add them here.
-         (Hence, don't publish them additionally!) -->
-	<joint name="camera_depth_joint" type="fixed">
-	  <origin xyz="0 0 0" rpy="0 0 0" />
-	  <parent link="camera_link" />
-	  <child link="camera_depth_frame" />
-	</joint>
-	<link name="camera_depth_frame"/>
-	<joint name="camera_depth_optical_joint" type="fixed">
-	  <origin xyz="0 0 0" rpy="0 0 0" />
-	  <parent link="camera_link" />
-	  <child link="camera_depth_optical_frame" />
-	</joint>
-	<link name="camera_depth_optical_frame"/>
-  <link name="laser">
-    <visual>
-      <geometry>
-        <box size="0.0762 0.0762 0.0762"/>
-      </geometry>
-      <material name="blue">
-	<color rgba="0.1 0.1 1 1"/>
-      </material>
-    </visual>
-    <!--<collision>
-      <geometry>
-        <box size="0.0762 0.2794 0.0762"/>
-      </geometry>
-    </collision>-->
-   <inertial>
-      <mass value="0.25"/>
-      <inertia ixx="1.0" iyy="1.0" izz="1.0"
-               ixy="0" ixz="0" iyz="0"/>
-    </inertial>
-  </link>
-  <joint name="laser_joint" type="fixed">
-    <axis xyz="0 0 1"/>
-    <parent link="body_link"/>
-    <child link="laser"/>
-    <origin rpy="0 0 0" xyz="0.0 0 0.75"/>
-  </joint>
-  <link name="pocketbot">
-    <visual>
-      <geometry>
-        <box size="0.1080 0.1920 0.005"/>
-      </geometry>
-      <material name="red">
-	<color rgba="0.1 0.1 1 1"/>
-      </material>
-    </visual>
-    <!--<collision>
-      <geometry>
-        <box size="0.0762 0.2794 0.0762"/>
-      </geometry>
-    </collision>-->
-   <inertial>
-      <mass value="0.25"/>
-      <inertia ixx="1.0" iyy="1.0" izz="1.0"
-               ixy="0" ixz="0" iyz="0"/>
-    </inertial>
-  </link>
-  <joint name="pocketbot_joint" type="continuous">
-    <axis xyz="0 0 1"/>
-    <parent link="body_link"/>
-    <child link="pocketbot"/>
-    <origin rpy="0 0 0" xyz="0.0 0.2 0.5"/>
-  </joint>
-  <link name="hitch_front_link">
-    <visual>
-      <geometry>
-        <cylinder length="0.1524" radius="0.01"/>
-      </geometry>
-      <material name="silver">
-	<color rgba="0.75 0.75 0.75 1"/>
-      </material>
-    </visual>
-    <collision>
-      <geometry>
-        <cylinder length="0.1524" radius="0.01"/>
-      </geometry>
-    </collision>
-    <inertial>
-      <mass value="0.1"/>
-      <inertia ixx="1.0" iyy="1.0" izz="1.0"
-               ixy="0" ixz="0" iyz="0"/>
-    </inertial>
-  </link>
-  <joint name="hitch_joint" type="fixed">
-    <axis xyz="0 0 1"/>
-    <parent link="base_link"/>
-    <child link="hitch_front_link"/>
-    <origin rpy="0 0 0" xyz="0.18 0 0.0762"/>
-  </joint>
-  <link name="wheel_front_left">
-    <visual>
-      <geometry>
-        <cylinder length="0.0508" radius="0.0762"/>
-      </geometry>
-      <material name="black">
-        <color rgba="0 0 0 1"/>
-      </material>
-    </visual>
-    <collision>
-      <geometry>
-        <cylinder length="0.0508" radius="0.0762"/>
-      </geometry>
-    </collision>
-    <inertial>
-      <mass value="0.1"/>
-      <inertia ixx="1.0" iyy="1.0" izz="1.0"
-               ixy="0" ixz="0" iyz="0"/>
-    </inertial>
-  </link>
-  <joint name="axis_front_left" type="continuous">
-    <axis xyz="0 0 1"/>
-    <parent link="base_link"/>
-    <child link="wheel_front_left"/>
-    <origin rpy="-1.5708 0 0" xyz="0.165862 0.18034 0"/>
-  </joint>
- <link name="wheel_front_right">
-    <visual>
-      <geometry>
-        <cylinder length="0.0508" radius="0.0762"/>
-      </geometry>
-      <material name="black"/>
-    </visual>
-    <collision>
-      <geometry>
-        <cylinder length="0.0508" radius="0.0762"/>
-      </geometry>
-    </collision>
-    <inertial>
-      <mass value="0.1"/>
-      <inertia ixx="1.0" iyy="1.0" izz="1.0"
-               ixy="0" ixz="0" iyz="0"/>
-    </inertial>
-  </link>
-  <joint name="axis_front_right" type="continuous">
-    <axis xyz="0 0 1"/>
-    <parent link="base_link"/>
-    <child link="wheel_front_right"/>
-    <origin rpy="-1.5708 0 0" xyz="0.165862 -0.18034 0"/>
-  </joint>
-  <link name="wheel_rear_right">
-    <visual>
-      <geometry>
-        <cylinder length="0.0508" radius="0.0762"/>
-      </geometry>
-      <material name="black"/>
-    </visual>
-    <collision>
-      <geometry>
-        <cylinder length="0.0508" radius="0.0762"/>
-      </geometry>
-    </collision>
-    <inertial>
-      <mass value="0.1"/>
-      <inertia ixx="1.0" iyy="1.0" izz="1.0"
-               ixy="0" ixz="0" iyz="0"/>
-    </inertial>
-  </link>
-  <joint name="axis_rear_right" type="continuous">
-    <axis xyz="0 0 1"/>
-    <parent link="base_link"/>
-    <child link="wheel_rear_right"/>
-    <origin rpy="-1.5708 0 0" xyz="-0.165862 -0.18034 0"/>
-  </joint>
-  <link name="wheel_rear_left">
-    <visual>
-      <geometry>
-        <cylinder length="0.0508" radius="0.0762"/>
-      </geometry>
-      <material name="black"/>
-    </visual>
-    <collision>
-      <geometry>
-        <cylinder length="0.0508" radius="0.0762"/>
-      </geometry>
-    </collision>
-    <inertial>
-      <mass value="0.1"/>
-      <inertia ixx="1.0" iyy="1.0" izz="1.0"
-               ixy="0" ixz="0" iyz="0"/>
-    </inertial>
-    <gazebo reference="wheel_rear_left">
-      <material>Gazebo/Black</material>
-    </gazebo>
-  </link>
-  <joint name="axis_rear_left" type="continuous">
-    <axis xyz="0 0 1"/>
-    <parent link="base_link"/>
-    <child link="wheel_rear_left"/>
-    <origin rpy="-1.5708 0 0" xyz="-0.165862 0.18034 0"/>
-  </joint>
-  <gazebo>
-    <plugin name="differential_drive_controller" filename="libgazebo_ros_diff_drive.so">
-      <alwaysOn>true</alwaysOn>
-      <updateRate>20</updateRate>
-      <leftJoint>axis_front_left</leftJoint>
-      <rightJoint>axis_front_right</rightJoint>
-      <wheelSeparation>0.254</wheelSeparation>
-      <wheelDiameter>0.1524</wheelDiameter>
-      <torque>20</torque>
-      <commandTopic>pocketbot/cmd_vel</commandTopic>
-      <odometryTopic>odom</odometryTopic>
-      <odometryFrame>odom</odometryFrame>
-      <robotBaseFrame>base_link</robotBaseFrame>
-    </plugin>
-  </gazebo>
-<!--<gazebo>
-  <plugin name="skid_steer_drive_controller" filename="libgazebo_ros_skid_steer_drive.so">
-    <updateRate>100.0</updateRate>
-    <robotNamespace></robotNamespace>
-    <leftFrontJoint>axis_front_left</leftFrontJoint>
-    <rightFrontJoint>axis_front_right</rightFrontJoint>
-    <leftRearJoint>axis_rear_left</leftRearJoint>
-    <rightRearJoint>axis_rear_right</rightRearJoint>
-    <wheelSeparation>0.254</wheelSeparation>
-    <wheelDiameter>0.1524</wheelDiameter>
-    <robotBaseFrame>base_link</robotBaseFrame>
-    <torque>10</torque>
-    <commandTopic>pocketbot/cmd_vel</commandTopic>
-    <broadcastTF>0</broadcastTF>
-    <odometryFrame>odom</odometryFrame>
-    <odometryTopic>odom</odometryTopic>
-  </plugin>
-</gazebo> -->
-  <!--<plugin name="joint_state_publisher" filename="libgazebo_ros_joint_state_publisher.so">
-    <jointName>axis_front_left, axis_front_right, axis_rear_left, axis_rear_right</jointName>
-    <updateRate>100</updateRate>
-  </plugin>-->
-<gazebo reference="laser">
-    <material>Gazebo/Blue</material>
-    <sensor type="ray" name="head_hokuyo_sensor">
-      <pose>0 0 0 0 0 0</pose>
-      <visualize>false</visualize>
-      <update_rate>40</update_rate>
-      <ray>
-        <scan>
-          <horizontal>
-            <samples>720</samples>
-            <resolution>1</resolution>
-            <min_angle>-1.570795</min_angle>
-            <max_angle>1.570795</max_angle>
-          </horizontal>
-        </scan>
-        <range>
-          <min>0.10</min>
-          <max>30.0</max>
-          <resolution>0.01</resolution>
-        </range>
-        <noise>
-          <type>gaussian</type>
-          <!-- Noise parameters based on published spec for Hokuyo laser
-               achieving "+-30mm" accuracy at range < 10m.  A mean of 0.0m and
-               stddev of 0.01m will put 99.7% of samples within 0.03m of the true
-               reading. -->
-          <mean>0.0</mean>
-          <stddev>0.01</stddev>
-        </noise>
-      </ray>
-      <plugin name="gazebo_ros_head_hokuyo_controller" filename="libgazebo_ros_laser.so">
-        <topicName>/scan</topicName>
-        <frameName>laser</frameName>
-      </plugin>
-    </sensor>
-  </gazebo>
-  <gazebo reference="camera_link">
-    <material>Gazebo/Blue</material>
-    <sensor type="depth" name="camera">
-        <always_on>true</always_on>
-        <update_rate>20.0</update_rate>
-        <visualize>true</visualize>
-        <camera>
-            <horizontal_fov>1.046666667</horizontal_fov>
-            <image>
-                <width>640</width>
-                <height>480</height>
-                <format>B8G8R8</format>
-            </image>
-            <depth_camera>
-            </depth_camera>
-            <clip>
-                <near>0.05</near>
-                <far>8.0</far>
-            </clip>
-        </camera>
-        <plugin name="kinect_camera_controller" filename="libgazebo_ros_openni_kinect.so">
-            <cameraName>camera</cameraName>
-            <alwaysOn>true</alwaysOn>
-            <updateRate>10.0</updateRate>
-            <frameName>camera_link</frameName>
-            <imageTopicName>rgb/image_rect_color</imageTopicName>
-            <depthImageTopicName>depth_registered/image_raw</depthImageTopicName>
-            <pointCloudTopicName>depth/points</pointCloudTopicName>
-            <cameraInfoTopicName>rgb/camera_info</cameraInfoTopicName>
-            <depthImageCameraInfoTopicName>depth/camera_info</depthImageCameraInfoTopicName>
-          <baseline>0.1</baseline>
-          <distortion_k1>0.0</distortion_k1>
-          <distortion_k2>0.0</distortion_k2>
-          <distortion_k3>0.0</distortion_k3>
-          <distortion_t1>0.0</distortion_t1>
-          <distortion_t2>0.0</distortion_t2>
-          <pointCloudCutoff>0.4</pointCloudCutoff>
-        </plugin>
-    </sensor>
-</gazebo>
 </robot>

Commit message: Added pi 3 setup in ansible

File: docker_ros_nodes/ros-mars-rover-description/model.urdf.xacro (robot description, xacro)
@@ -22,3 +22,289 @@
     </inertial>
   </link>
+  <gazebo reference="base_link">
+    <material>Gazebo/Black</material>
+  </gazebo>
+  <link name="body_link">
+    <visual>
+      <geometry>
+        <cylinder length="1.04775" radius="0.2032"/>
+        <!-- <mesh filename="http://localhost:8888/rover.stl" scale="0.015 0.015 0.015"/> -->
+      </geometry>
+      <!-- <material name="clear">
+        <color rgba="0.75 0.75 0.75 0.4"/>
+      </material> -->
+      <material name="clear">
+        <color rgba="0.75 0.5 1.0 1.0"/>
+      </material>
+    </visual>
+    <!--<collision>
+      <geometry>
+        <cylinder length="1.04775" radius="0.2032"/>
+      </geometry>
+    </collision>-->
+    <inertial>
+      <mass value="10.0"/>
+      <inertia ixx="1.0" iyy="1.0" izz="1.0"
+               ixy="0" ixz="0" iyz="0"/>
+    </inertial>
+  </link>
+  <joint name="center_joint" type="fixed">
+    <axis xyz="0 0 1"/>
+    <parent link="base_link"/>
+    <child link="body_link"/>
+    <origin rpy="0 0 0" xyz="0 0 0.551815"/>
+  </joint>
+  <link name="camera_link">
+    <visual>
+      <origin rpy="0 0 0"/>
+      <geometry>
+        <box size="0.0762 0.2794 0.0762"/>
+      </geometry>
+      <material name="red">
+	<color rgba="1 0.1 0.1 1"/>
+      </material>
+    </visual>
+    <!--<collision>
+      <geometry>
+        <box size="0.0762 0.2794 0.0762"/>
+      </geometry>
+    </collision>-->
+   <inertial>
+      <mass value="0.25"/>
+      <inertia ixx="1.0" iyy="1.0" izz="1.0"
+               ixy="0" ixz="0" iyz="0"/>
+    </inertial>
+  </link>
+  <joint name="camera_joint" type="fixed">
+    <axis xyz="0 0 0"/>
+    <parent link="body_link"/>
+    <child link="camera_link"/>
+    <origin rpy="0 0 0" xyz="0.15 0 -0.25"/>
+  </joint>
+    <!-- The fixed joints & links below are usually published by static_transformers launched by the OpenNi launch
+         files. However, for Gazebo simulation we need them, so we add them here.
+         (Hence, don't publish them additionally!) -->
+	<joint name="camera_depth_joint" type="fixed">
+	  <origin xyz="0 0 0" rpy="0 0 0" />
+	  <parent link="camera_link" />
+	  <child link="camera_depth_frame" />
+	</joint>
+	<link name="camera_depth_frame"/>
+	<joint name="camera_depth_optical_joint" type="fixed">
+	  <origin xyz="0 0 0" rpy="0 0 0" />
+	  <parent link="camera_link" />
+	  <child link="camera_depth_optical_frame" />
+	</joint>
+	<link name="camera_depth_optical_frame"/>
+  <link name="wheel_front_left">
+    <visual>
+      <geometry>
+        <cylinder length="0.0508" radius="0.0762"/>
+      </geometry>
+      <material name="black">
+        <color rgba="0 0 0 1"/>
+      </material>
+    </visual>
+    <collision>
+      <geometry>
+        <cylinder length="0.0508" radius="0.0762"/>
+      </geometry>
+    </collision>
+    <inertial>
+      <mass value="0.1"/>
+      <inertia ixx="1.0" iyy="1.0" izz="1.0"
+               ixy="0" ixz="0" iyz="0"/>
+    </inertial>
+  </link>
+  <joint name="axis_front_left" type="continuous">
+    <axis xyz="0 0 1"/>
+    <parent link="base_link"/>
+    <child link="wheel_front_left"/>
+    <origin rpy="-1.5708 0 0" xyz="0.165862 0.18034 0"/>
+  </joint>
+ <link name="wheel_front_right">
+    <visual>
+      <geometry>
+        <cylinder length="0.0508" radius="0.0762"/>
+      </geometry>
+      <material name="black"/>
+    </visual>
+    <collision>
+      <geometry>
+        <cylinder length="0.0508" radius="0.0762"/>
+      </geometry>
+    </collision>
+    <inertial>
+      <mass value="0.1"/>
+      <inertia ixx="1.0" iyy="1.0" izz="1.0"
+               ixy="0" ixz="0" iyz="0"/>
+    </inertial>
+  </link>
+  <joint name="axis_front_right" type="continuous">
+    <axis xyz="0 0 1"/>
+    <parent link="base_link"/>
+    <child link="wheel_front_right"/>
+    <origin rpy="-1.5708 0 0" xyz="0.165862 -0.18034 0"/>
+  </joint>
+  <link name="wheel_rear_right">
+    <visual>
+      <geometry>
+        <cylinder length="0.0508" radius="0.0762"/>
+      </geometry>
+      <material name="black"/>
+    </visual>
+    <collision>
+      <geometry>
+        <cylinder length="0.0508" radius="0.0762"/>
+      </geometry>
+    </collision>
+    <inertial>
+      <mass value="0.1"/>
+      <inertia ixx="1.0" iyy="1.0" izz="1.0"
+               ixy="0" ixz="0" iyz="0"/>
+    </inertial>
+  </link>
+  <joint name="axis_rear_right" type="continuous">
+    <axis xyz="0 0 1"/>
+    <parent link="base_link"/>
+    <child link="wheel_rear_right"/>
+    <origin rpy="-1.5708 0 0" xyz="-0.165862 -0.18034 0"/>
+  </joint>
+  <link name="wheel_rear_left">
+    <visual>
+      <geometry>
+        <cylinder length="0.0508" radius="0.0762"/>
+      </geometry>
+      <material name="black"/>
+    </visual>
+    <collision>
+      <geometry>
+        <cylinder length="0.0508" radius="0.0762"/>
+      </geometry>
+    </collision>
+    <inertial>
+      <mass value="0.1"/>
+      <inertia ixx="1.0" iyy="1.0" izz="1.0"
+               ixy="0" ixz="0" iyz="0"/>
+    </inertial>
+    <gazebo reference="wheel_rear_left">
+      <material>Gazebo/Black</material>
+    </gazebo>
+  </link>
+  <joint name="axis_rear_left" type="continuous">
+    <axis xyz="0 0 1"/>
+    <parent link="base_link"/>
+    <child link="wheel_rear_left"/>
+    <origin rpy="-1.5708 0 0" xyz="-0.165862 0.18034 0"/>
+  </joint>
+  <gazebo>
+    <plugin name="differential_drive_controller" filename="libgazebo_ros_diff_drive.so">
+      <alwaysOn>true</alwaysOn>
+      <updateRate>20</updateRate>
+      <leftJoint>axis_front_left</leftJoint>
+      <rightJoint>axis_front_right</rightJoint>
+      <wheelSeparation>0.254</wheelSeparation>
+      <wheelDiameter>0.1524</wheelDiameter>
+      <torque>20</torque>
+      <commandTopic>pocketbot/cmd_vel</commandTopic>
+      <odometryTopic>odom</odometryTopic>
+      <odometryFrame>map</odometryFrame>
+      <robotBaseFrame>base_link</robotBaseFrame>
+      <legacyMode>false</legacyMode>
+    </plugin>
+  </gazebo>
+<!--<gazebo>
+  <plugin name="skid_steer_drive_controller" filename="libgazebo_ros_skid_steer_drive.so">
+    <updateRate>100.0</updateRate>
+    <robotNamespace></robotNamespace>
+    <leftFrontJoint>axis_front_left</leftFrontJoint>
+    <rightFrontJoint>axis_front_right</rightFrontJoint>
+    <leftRearJoint>axis_rear_left</leftRearJoint>
+    <rightRearJoint>axis_rear_right</rightRearJoint>
+    <wheelSeparation>0.254</wheelSeparation>
+    <wheelDiameter>0.1524</wheelDiameter>
+    <robotBaseFrame>base_link</robotBaseFrame>
+    <torque>10</torque>
+    <commandTopic>pocketbot/cmd_vel</commandTopic>
+    <broadcastTF>0</broadcastTF>
+    <odometryFrame>odom</odometryFrame>
+    <odometryTopic>odom</odometryTopic>
+  </plugin>
+</gazebo> -->
+  <!--<plugin name="joint_state_publisher" filename="libgazebo_ros_joint_state_publisher.so">
+    <jointName>axis_front_left, axis_front_right, axis_rear_left, axis_rear_right</jointName>
+    <updateRate>100</updateRate>
+  </plugin>-->
+<gazebo reference="laser">
+    <material>Gazebo/Blue</material>
+    <sensor type="ray" name="head_hokuyo_sensor">
+      <pose>0 0 0 0 0 0</pose>
+      <visualize>false</visualize>
+      <update_rate>40</update_rate>
+      <ray>
+        <scan>
+          <horizontal>
+            <samples>720</samples>
+            <resolution>1</resolution>
+            <min_angle>-1.570795</min_angle>
+            <max_angle>1.570795</max_angle>
+          </horizontal>
+        </scan>
+        <range>
+          <min>0.10</min>
+          <max>30.0</max>
+          <resolution>0.01</resolution>
+        </range>
+        <noise>
+          <type>gaussian</type>
+          <mean>0.0</mean>
+          <stddev>0.01</stddev>
+        </noise>
+      </ray>
+      <plugin name="gazebo_ros_head_hokuyo_controller" filename="libgazebo_ros_laser.so">
+        <topicName>/scan</topicName>
+        <frameName>laser</frameName>
+      </plugin>
+    </sensor>
+  </gazebo>
+  <gazebo reference="camera_link">
+    <material>Gazebo/Blue</material>
+    <sensor type="depth" name="camera">
+        <always_on>true</always_on>
+        <update_rate>20.0</update_rate>
+        <visualize>true</visualize>
+        <camera>
+            <horizontal_fov>1.046666667</horizontal_fov>
+            <image>
+                <width>640</width>
+                <height>480</height>
+                <format>B8G8R8</format>
+            </image>
+            <depth_camera>
+            </depth_camera>
+            <clip>
+                <near>0.05</near>
+                <far>8.0</far>
+            </clip>
+        </camera>
+        <plugin name="kinect_camera_controller" filename="libgazebo_ros_openni_kinect.so">
+            <cameraName>camera</cameraName>
+            <alwaysOn>true</alwaysOn>
+            <updateRate>10.0</updateRate>
+            <frameName>camera_link</frameName>
+            <imageTopicName>rgb/image_rect_color</imageTopicName>
+            <depthImageTopicName>depth_registered/image_raw</depthImageTopicName>
+            <pointCloudTopicName>depth/points</pointCloudTopicName>
+            <cameraInfoTopicName>rgb/camera_info</cameraInfoTopicName>
+            <depthImageCameraInfoTopicName>depth/camera_info</depthImageCameraInfoTopicName>
+          <baseline>0.1</baseline>
+          <distortion_k1>0.0</distortion_k1>
+          <distortion_k2>0.0</distortion_k2>
+          <distortion_k3>0.0</distortion_k3>
+          <distortion_t1>0.0</distortion_t1>
+          <distortion_t2>0.0</distortion_t2>
+          <pointCloudCutoff>0.4</pointCloudCutoff>
+        </plugin>
+    </sensor>
+</gazebo>
 </robot>
